File: hardware/CAN_Power_Velleman/CAN_Power.sch (KiCad schematic (older format))
At the start: 11 parts, among them K1 CONN_3, K2 CONN_3, P1 CONN_1, P2 CONN_1, P3 CONN_1, P5 CONN_4, P6 CONN_1, P7 CONN_1, P8 CONN_1, P9 FUSE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

Commit message: Connected PE to GND
Connections:
- net GNDPWR is gone; now on net GND: K2.1 (P1), U1.17 (Shield), U1.18 (Shield)
Changed lines of the file:
@@
 Sheet 1 1
 Title ""
-Date "28 oct 2014"
+Date "17 nov 2014"
 Rev ""
 Comp ""
@@
 	5900 5900 5900 6050
 Wire Wire Line
-	6500 5850 6200 5850
+	6200 5850 6750 5850
 Connection ~ 6200 5850
 Wire Wire Line
 	4350 2500 4350 7050
 Wire Wire Line
-	4350 7050 6500 7050
+	4350 7050 6750 7050
 Connection ~ 6500 6400
 Wire Wire Line
@@
 Wire Wire Line
 	5350 2500 4350 2500
+Wire Wire Line
+	6750 7050 6750 5850
+Connection ~ 6500 7050
+Connection ~ 6500 5850
 $EndSCHEMATC
