File: avr/AT90CAN32_Latching_Relay/hardware/Latching_Relay.sch (KiCad schematic (older format))
At the start: 25 parts, among them K1 CONN_3, K2 CONN_3, P1 CONN_3X2, Q1 BC237, Q2 BC237, SW1 SW_PUSH, U1 RELAY_BISTABLE, U2 AT90CAN32, U3 7805, U4 MCP2551, U6 RJ45_DUAL, X1 16MHz

Commit message: Schematic and PCB finalized
Parts:
- removed D2, D3: DIODE, symbol DIODE
- removed Q1, Q2: BC237, TO92-EBC, symbol BC237
- removed R3, R4: 300, symbol R
- added U2: ULN2003A, symbol ULN2003A
- U1: footprint (none) -> ~
- renumbered C5 to C4, C6 to C5, C4 to C6, K2 to K1, K1 to K2, U2 to U3, U3 to U4, U4 to U5
Connections:
- net +5V: now also U1.3 (A3), U2.9 (COM)
- net GND: now also U2.8 (GND); no longer U1.3 (A3)
- net at U3.35 (PC0(A8)): now also U2.1 (I1)
- net at U3.36 (PC1(A9)): now also U2.2 (I2)
- net at U1.2 (A2): now also U2.15 (O2)
- net at U1.1 (A1): now also U2.16 (O1)
- no-connect marks 48 -> 61
Changed lines of the file:
@@
 LIBS:valves
 LIBS:Molex_Dual_RJ45
+LIBS:Relay
 LIBS:Latching_Relay-cache
 EELAYER 27 0
@@
 Sheet 1 1
 Title ""
-Date "25 mar 2015"
+Date "30 mar 2015"
 Rev ""
 Comp ""
@@
 NoConn ~ 8250 3550
 $Comp
-L MCP2551 U4
+L MCP2551 U5
 U 1 1 52152F80
 P 7700 3300
-F 0 "U4" H 7700 3150 60  0000 C CNN
+F 0 "U5" H 7700 3150 60  0000 C CNN
 F 1 "MCP2551" H 7700 2600 60  0000 C CNN
 F 2 "" H 7700 3300 60  0001 C CNN
@@
 $EndComp
 $Comp
-L AT90CAN32 U2
+L AT90CAN32 U3
 U 1 1 52152F75
 P 5450 2850
-F 0 "U2" H 5600 3600 60  0000 C CNN
+F 0 "U3" H 5600 3600 60  0000 C CNN
 F 1 "AT90CAN32" H 5250 2500 60  0000 C CNN
 F 2 "" H 5450 2850 60  0001 C CNN
@@
 PD1
 $Comp
-L 7805 U3
+L 7805 U4
 U 1 1 52BC76CC
 P 7700 1300
-F 0 "U3" H 7850 1104 60  0000 C CNN
+F 0 "U4" H 7850 1104 60  0000 C CNN
 F 1 "7805" H 7700 1500 60  0000 C CNN
 F 2 "" H 7700 1300 60  0000 C CNN
@@
 $EndComp
 $Comp
-L C C4
+L C C6
 U 1 1 52BC77D5
 P 8100 1500
-F 0 "C4" H 8150 1600 50  0000 L CNN
+F 0 "C6" H 8150 1600 50  0000 L CNN
 F 1 "0.33uF" H 8150 1400 50  0000 L CNN
 F 2 "" H 8100 1500 60  0000 C CNN
@@
 $EndComp
 $Comp
-L CONN_3 K1
+L CONN_3 K2
 U 1 1 544570D5
 P 7500 2550
-F 0 "K1" V 7450 2550 50  0000 C CNN
+F 0 "K2" V 7450 2550 50  0000 C CNN
 F 1 "CONN_3" V 7550 2550 40  0000 C CNN
 F 2 "" H 7500 2550 60  0000 C CNN
@@
 NoConn ~ 4550 3300
 $Comp
-L C C5
+L C C4
 U 1 1 544964C0
 P 6050 1800
-F 0 "C5" H 6100 1900 50  0000 L CNN
+F 0 "C4" H 6100 1900 50  0000 L CNN
 F 1 "100nF" H 6100 1700 50  0000 L CNN
 F 2 "" H 6050 1800 60  0000 C CNN
@@
 $EndComp
 $Comp
-L C C6
+L C C5
 U 1 1 544966BB
 P 6300 6100
-F 0 "C6" H 6350 6200 50  0000 L CNN
+F 0 "C5" H 6350 6200 50  0000 L CNN
 F 1 "100nF" H 6350 6000 50  0000 L CNN
 F 2 "" H 6300 6100 60  0000 C CNN
@@
 NoConn ~ 9750 5100
 NoConn ~ 9750 3000
-$Comp
-L R R4
-U 1 1 5511C928
-P 3650 2300
-F 0 "R4" H 3730 2300 50  0000 C CNN
-F 1 "300" V 3650 2300 50  0000 C CNN
-F 2 "" H 3650 2300 60  0001 C CNN
-F 3 "" H 3650 2300 60  0001 C CNN
-	1    3650 2300
-	1    0    0    -1
-$EndComp
-$Comp
-L R R3
-U 1 1 5511C93D
-P 3300 2300
-F 0 "R3" H 3380 2300 50  0000 C CNN
-F 1 "300" V 3300 2300 50  0000 C CNN
-F 2 "" H 3300 2300 60  0001 C CNN
-F 3 "" H 3300 2300 60  0001 C CNN
-	1    3300 2300
-	1    0    0    -1
-$EndComp
 Wire Wire Line
 	4550 4150 3950 4150
@@
 	3950 2850 3650 2850
 Wire Wire Line
-	3650 2850 3650 2550
+	3650 2850 3650 900
 Wire Wire Line
 	4550 4250 3900 4250
@@
 	3900 2900 3300 2900
 Wire Wire Line
-	3300 2900 3300 2550
-$Comp
-L BC237 Q1
-U 1 1 5511CA67
-P 2800 1200
-F 0 "Q1" H 3000 1100 50  0000 C CNN
-F 1 "BC237" H 3050 1350 50  0000 C CNN
-F 2 "TO92-EBC" H 2990 1200 30  0001 C CNN
-F 3 "" H 2800 1200 60  0000 C CNN
-	1    2800 1200
-	-1   0    0    1
-$EndComp
-$Comp
-L BC237 Q2
-U 1 1 5511CA7E
-P 2800 1750
-F 0 "Q2" H 3000 1650 50  0000 C CNN
-F 1 "BC237" H 3050 1900 50  0000 C CNN
-F 2 "TO92-EBC" H 2990 1750 30  0001 C CNN
-F 3 "" H 2800 1750 60  0000 C CNN
-	1    2800 1750
-	-1   0    0    1
-$EndComp
-Wire Wire Line
-	3300 2050 3300 1750
-Wire Wire Line
-	3300 1750 3000 1750
-Wire Wire Line
-	3650 2050 3650 1200
-Wire Wire Line
-	3650 1200 3000 1200
-$Comp
-L +5V #PWR014
-U 1 1 5511CB9E
-P 3200 950
-F 0 "#PWR014" H 3200 1040 20  0001 C CNN
-F 1 "+5V" H 3200 1040 30  0000 C CNN
-F 2 "" H 3200 950 60  0001 C CNN
-F 3 "" H 3200 950 60  0001 C CNN
-	1    3200 950
-	1    0    0    -1
-$EndComp
-Wire Wire Line
-	2700 1950 3200 1950
-Wire Wire Line
-	3200 1950 3200 950
-Wire Wire Line
-	2700 1400 3200 1400
-Connection ~ 3200 1400
-$Comp
-L RELAY_BISTABLE U1
-U 1 1 5511D3E6
-P 1650 3100
-F 0 "U1" H 1650 3100 60  0000 C CNN
-F 1 "RELAY_BISTABLE" H 1650 2850 60  0000 C CNN
-F 2 "" H 1650 3100 60  0000 C CNN
-F 3 "" H 1650 3100 60  0000 C CNN
-	1    1650 3100
-	0    1    1    0
-$EndComp
-Wire Wire Line
-	2700 1550 1800 1550
-Wire Wire Line
-	1800 1550 1800 2200
-Wire Wire Line
-	2700 1000 1400 1000
-Wire Wire Line
-	1400 1000 1400 2200
-$Comp
-L GND #PWR015
+	3300 2900 3300 1000
+$Comp
+L GND #PWR014
 U 1 1 5511D527
-P 2300 2650
-F 0 "#PWR015" H 2300 2650 30  0001 C CNN
-F 1 "GND" H 2300 2580 30  0001 C CNN
-F 2 "" H 2300 2650 60  0001 C CNN
-F 3 "" H 2300 2650 60  0001 C CNN
-	1    2300 2650
-	1    0    0    -1
-$EndComp
-Wire Wire Line
-	1600 2200 1600 1950
-Wire Wire Line
-	1600 1950 2300 1950
-Wire Wire Line
-	2300 1950 2300 2650
-$Comp
-L DIODE D2
-U 1 1 5511D5C8
-P 1050 1850
-F 0 "D2" H 1050 1950 40  0000 C CNN
-F 1 "DIODE" H 1050 1750 40  0000 C CNN
-F 2 "" H 1050 1850 60  0000 C CNN
-F 3 "" H 1050 1850 60  0000 C CNN
-	1    1050 1850
-	0    -1   -1   0
-$EndComp
-Wire Wire Line
-	1050 1650 1050 1350
-Wire Wire Line
-	1050 1350 1400 1350
-Connection ~ 1400 1350
-Wire Wire Line
-	1050 2050 1050 2100
-Wire Wire Line
-	1050 2100 2100 2100
-Connection ~ 1600 2100
-$Comp
-L DIODE D3
-U 1 1 5511D718
-P 2100 1850
-F 0 "D3" H 2100 1950 40  0000 C CNN
-F 1 "DIODE" H 2100 1750 40  0000 C CNN
-F 2 "" H 2100 1850 60  0000 C CNN
-F 3 "" H 2100 1850 60  0000 C CNN
-	1    2100 1850
-	0    -1   -1   0
-$EndComp
-Wire Wire Line
-	2100 1550 2100 1650
-Connection ~ 2100 1550
-Wire Wire Line
-	2100 2100 2100 2050
-$Comp
-L CONN_3 K2
+P 2600 1950
+F 0 "#PWR014" H 2600 1950 30  0001 C CNN
+F 1 "GND" H 2600 1880 30  0001 C CNN
+F 2 "" H 2600 1950 60  0001 C CNN
+F 3 "" H 2600 1950 60  0001 C CNN
+	1    2600 1950
+	1    0    0    -1
+$EndComp
+$Comp
+L CONN_3 K1
 U 1 1 5511D864
 P 1500 4450
-F 0 "K2" V 1450 4450 50  0000 C CNN
+F 0 "K1" V 1450 4450 50  0000 C CNN
 F 1 "CONN_3" V 1550 4450 40  0000 C CNN
 F 2 "" H 1500 4450 60  0000 C CNN
@@
 	9400 4300 8400 4300
 Connection ~ 8400 4300
+$Comp
+L RELAY_BISTABLE U1
+U 1 1 55147B82
+P 1650 3100
+F 0 "U1" H 1650 3100 60  0000 C CNN
+F 1 "RELAY_BISTABLE" H 1650 2850 60  0000 C CNN
+F 2 "~" H 1650 3100 60  0000 C CNN
+F 3 "~" H 1650 3100 60  0000 C CNN
+	1    1650 3100
+	0    1    1    0
+$EndComp
+NoConn ~ 2250 3350
+NoConn ~ 2250 3500
+NoConn ~ 2250 3650
+$Comp
+L ULN2003A U2
+U 1 1 5515B38B
+P 2250 1300
+F 0 "U2" H 2250 1400 70  0000 C CNN
+F 1 "ULN2003A" H 2250 1200 70  0000 C CNN
+F 2 "" H 2250 1300 60  0000 C CNN
+F 3 "" H 2250 1300 60  0000 C CNN
+	1    2250 1300
+	-1   0    0    -1
+$EndComp
+$Comp
+L +5V #PWR015
+U 1 1 5515B56A
+P 1450 1700
+F 0 "#PWR015" H 1450 1790 20  0001 C CNN
+F 1 "+5V" H 1450 1790 30  0000 C CNN
+F 2 "" H 1450 1700 60  0001 C CNN
+F 3 "" H 1450 1700 60  0001 C CNN
+	1    1450 1700
+	1    0    0    -1
+$EndComp
+Wire Wire Line
+	1600 1700 1450 1700
+Wire Wire Line
+	2600 1950 2600 1800
+Wire Wire Line
+	3650 900  2900 900
+Wire Wire Line
+	3300 1000 2900 1000
+Wire Wire Line
+	1600 1700 1600 2200
+Connection ~ 2600 1900
+Wire Wire Line
+	1600 900  1300 900
+Wire Wire Line
+	1300 900  1300 2000
+Wire Wire Line
+	1300 2000 1800 2000
+Wire Wire Line
+	1800 2000 1800 2200
+Wire Wire Line
+	1600 1000 1400 1000
+Wire Wire Line
+	1400 1000 1400 2200
+NoConn ~ 1600 1100
+NoConn ~ 1600 1200
+NoConn ~ 1600 1300
+NoConn ~ 1600 1400
+NoConn ~ 1600 1500
+NoConn ~ 2900 1100
+NoConn ~ 2900 1200
+NoConn ~ 2900 1300
+NoConn ~ 2900 1500
+NoConn ~ 2900 1400
 $EndSCHEMATC
