File: avr/AT90CAN32_Latching_Relay/hardware/Latching_Relay.kicad_pcb (KiCad board)
At the start: 2 copper layers, 24 parts, among them K1 CONN_3, P1 CONN_3X2, SW1 SW_PUSH, U1 DS1820, U2 AT90CAN32, U3 7805, U4 MCP2551, U5 HIH4000, U6 RJ45_DUAL, X1 16MHz

Commit message: Schematic and PCB finalized
Parts:
- removed the 1PIN at (191.0, 80.0)
- removed the 1PIN at (146.0, 80.0)
- removed the 1PIN at (146.0, 144.0)
- removed the 1PIN at (191.0, 144.0)
- removed R3: 470k, SM1206
- added 1PIN: P***, 1pin, F.Cu at (238.0, 151.0)
- added 1PIN: P***, 1pin, F.Cu at (199.0, 151.0)
- added 1PIN: P***, 1pin, F.Cu at (238.0, 73.0)
- added 1PIN: P***, 1pin, F.Cu at (199.0, 73.0)
- added K2: CONN_3, PIN_ARRAY_3X1, F.Cu at (223.7, 126.5)
- C4: value 0.33uF -> 100nF
- C6: value 100nF -> 0.33uF
- K1: footprint PIN_ARRAY_3X1 -> bornier3
- U1: value DS1820 -> RELAY_BISTABLE; footprint PIN_ARRAY_3X1 -> PCB relay bistable
- U2: value AT90CAN32 -> ULN2003A; footprint TQFP64_08 -> SO16E
- U3: value 7805 -> AT90CAN32; footprint SOT223 -> TQFP64_08
- U4: value MCP2551 -> 7805; footprint SO8E -> SOT223
- U5: value HIH4000 -> MCP2551; footprint PIN_ARRAY_3X1 -> SO8E
- moved C5 81.2 mm to (233.9, 134.1)
- moved U5 79.4 mm to (224.9, 133.7), turned to 270 degrees
- moved C6 74.7 mm to (230.7, 134.1), turned to 270 degrees
- moved K1 59.6 mm to (217.9, 72.4), turned to 180 degrees
- moved R1 59.3 mm to (211.8, 124.1), turned to 90 degrees
- moved D1 54.8 mm to (232.3, 109.8), turned to 180 degrees
- moved P1 54.8 mm to (203.1, 110.9)
- moved R2 54.7 mm to (232.3, 106.0)
- moved U4 54.3 mm to (231.6, 124.7), turned to 0 degrees
- moved C2 53.9 mm to (219.7, 124.0)
- moved SW1 53.4 mm to (231.4, 97.7)
- moved C1 53.3 mm to (215.4, 124.1)
- moved U6 51.7 mm to (218.6, 140.8)
- moved X1 50.5 mm to (212.2, 131.0)
- moved C3 44.1 mm to (222.6, 99.1), turned to 180 degrees
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Connections:
- C1 pad 2: N-0000023 -> N-0000040
- C2 pad 2: N-0000024 -> N-0000041
- C4 pad 1: +12V -> +5V
- C5 pad 1: +5V -> GND
- C5 pad 2: GND -> +5V
- C6 pad 1: GND -> +12V
- C6 pad 2: +5V -> GND
- D1 pad 1: N-0000018 -> N-0000075
- D1 pad 2: N-0000011 -> N-000004
- K1 pad 1: GND -> N-0000027
- K1 pad 2: N-0000016 -> N-0000038
- K1 pad 3: N-0000017 -> N-0000037
- P1 pad 3: N-000005 -> N-000008
- P1 pad 5: N-0000010 -> N-000009
- R1 pad 2: N-0000010 -> N-000009
- R2 pad 2: N-0000011 -> N-0000075
- SW1 pad 1: N-0000015 -> N-000003
- U1 pad 1: GND -> N-0000028
- U1 pad 2: N-0000021 -> N-0000029
- U2 pad 1: (no net) -> N-0000023
- U2 pad 11: N-000005 -> (no net)
- U2 pad 15: (no net) -> N-0000029
- U2 pad 16: (no net) -> N-0000028
- U2 pad 2: /PD1 -> N-0000022
- U2 pad 3: /PE1 -> (no net)
- U2 pad 8: (no net) -> GND
- U2 pad 9: (no net) -> +5V
- U3 pad 1: +12V -> (no net)
- U3 pad 2: GND -> /PD1
- U3 pad 3: +5V -> /PE1
- U4 pad 1: N-000001 -> +12V
- U4 pad 4: N-000002 -> (no net)
- U5 pad 1: GND -> N-000006
- U5 pad 2: N-0000020 -> GND
- U6 pad 12: N-0000014 -> N-0000035
- U6 pad 13: N-000006 -> N-0000034
- U6 pad 4: N-0000014 -> N-0000035
- U6 pad 5: N-000006 -> N-0000034
- X1 pad 1: N-0000024 -> N-0000041
- X1 pad 2: N-0000023 -> N-0000040
Routing:
- net GND: track 109.9 -> 205.2 mm, vias 8 -> 15
- net +5V: track 160.5 -> 203.9 mm, vias 0 -> 3
- net N-0000014: track 35.5 -> 0.00 mm
- net N-0000028: track 0.00 -> 28.9 mm
- net N-0000034: track 0.00 -> 28.8 mm
- net N-0000035: track 0.00 -> 27.8 mm
- net N-0000022: track 0.00 -> 26.4 mm, vias 0 -> 2
- net N-0000010: track 21.4 -> 0.00 mm
- net N-0000037: track 0.00 -> 21.3 mm
- net N-0000038: track 0.00 -> 21.1 mm
- net N-0000027: track 0.00 -> 20.9 mm
- net N-0000040: track 0.00 -> 19.5 mm
- net N-000007: track 0.00 -> 19.4 mm
- net N-000009: track 0.00 -> 18.6 mm
- net N-000006: track 33.7 -> 15.7 mm
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Other:
- board outline added: 44.7 x 87.1 mm
- net class Default: clearance 0.3 -> 0.254; trace_width 0.45 -> 0.254; via_dia 1.8 -> 0.889; via_drill 1 -> 0.635
- rule trace_clearance: 0.3 -> 0.254
- board text added: "VSCP LATCHING_RELAY"
- board text removed: "VSCP TEMP_HUMID"

Commit message: testing push from the office
Parts:
- moved U1 1.06 mm to (213.7, 80.8)
Routing:
- net +5V: track 203.9 -> 189.4 mm, vias 3 -> 4
- net N-0000037: track 21.3 -> 23.3 mm
- net N-0000029: track 17.7 -> 16.2 mm
- net N-0000027: track 20.9 -> 22.2 mm
- net N-0000038: track 21.1 -> 22.4 mm
